File: src/kicad/mm_2EQ_modern.kicad_pcb (KiCad board)
At the start: 2 copper layers, 44.5 x 21.6 mm, 24 parts, among them P1 In, P10 Gnd, P2 High, P3 Low, P4 Out, P9 +9V, U1 TLC2262

Commit message: routing second pass
Parts:
- moved C6 0.76 mm to (158.0, 61.7)
- moved P3 0.51 mm to (167.4, 46.5)
- moved R5 0.25 mm to (160.0, 50.0)
- moved C3 0.25 mm to (150.4, 55.4)
- moved R6 0.25 mm to (160.0, 52.6)
- moved R7 0.25 mm to (160.0, 55.1)
- moved R8 0.25 mm to (160.0, 57.7)
Routing:
- net ref: track 40.6 -> 55.8 mm
- net Net-(C9-Pad1): track 0.75 -> 5.49 mm
- net Net-(C3-Pad1): track 40.2 -> 42.9 mm
- net Net-(C3-Pad2): track 34.4 -> 36.6 mm
- net Net-(C5-Pad2): track 20.9 -> 22.0 mm
- added copper zone on F.Cu, net GND
Other:
- board size 44.5 x 21.6 mm -> 44.2 x 21.6 mm
- net class Default: clearance 0.508 -> 0.381
- rule trace_clearance: 0.508 -> 0.381
- board text added: "MM 2EQ modern"
- board text added: "bass"
- board text added: "treble"
- board text added: "v 1.0"
- board text added: "www.dolganoff.com/fr"
- board text removed: "MM 2EQ"
